Commit message: Change CITrack to models
Signed-off-by: Timo Korthals <tkorthals@cit-ec.uni-bielefeld.de>

File: urdf/cameras.xacro (robot description, xacro)
@@ -5,13 +5,13 @@
   <xacro:property name="PI_2" value="${PI / 2}"/>
   <link name="${map_frame}"/>
-  <xacro:include filename="$(find twb_gazebo)/urdf/jai-sp-5000m.xacro"/>
+  <xacro:include filename="$(find models)/urdf/jai-sp-5000m.xacro"/>
   <xacro:cam name="cam1_2" parent="${map_frame}" xyz="1.5 4.5 3.8" rpy="0 ${PI_2} ${PI}"/>
-  <xacro:include filename="$(find twb_gazebo)/urdf/jai-sp-5000m.xacro"/>
+  <xacro:include filename="$(find models)/urdf/jai-sp-5000m.xacro"/>
   <xacro:cam name="cam2_2" parent="${map_frame}" xyz="1.5 1.5 3.8" rpy="0 ${PI_2} ${PI}"/>
-  <xacro:include filename="$(find twb_gazebo)/urdf/jai-sp-5000m.xacro"/>
+  <xacro:include filename="$(find models)/urdf/jai-sp-5000m.xacro"/>
   <xacro:cam name="cam3_2" parent="${map_frame}" xyz="4.5 1.5 3.8" rpy="0 ${PI_2} ${PI}"/>
-  <xacro:include filename="$(find twb_gazebo)/urdf/jai-sp-5000m.xacro"/>
+  <xacro:include filename="$(find models)/urdf/jai-sp-5000m.xacro"/>
   <xacro:cam name="cam4_2" parent="${map_frame}" xyz="4.5 4.5 3.8" rpy="0 ${PI_2} ${PI_2}"/>
-  <xacro:include filename="$(find twb_gazebo)/urdf/jai-sp-5000c.xacro"/>
+  <xacro:include filename="$(find models)/urdf/jai-sp-5000c.xacro"/>
   <xacro:cam name="cam5_2" parent="${map_frame}" xyz="3.0 3.0 3.8" rpy="0 ${PI_2} ${PI}"/>
   <gazebo>

File: urdf/office_desk_models.xacro (robot description, xacro)
@@ -28,5 +28,5 @@
   <!--BALL PEN-->
   <xacro:property name="ball_pen" value="ball_pen"/>
-  <xacro:property name="ball_pen_model" value="package://twb_gazebo/meshes/ball_pen/meshes/ball_pen.dae"/>
+  <xacro:property name="ball_pen_model" value="package://models/meshes/ball_pen/meshes/ball_pen.dae"/>
   <joint name="${name}_${ball_pen}_joint" type="fixed">
     <axis xyz="0 0 1"/>
@@ -54,5 +54,5 @@
   <!--COMPUTER MOUSE-->
   <xacro:property name="computer_mouse" value="computer_mouse"/>
-  <xacro:property name="computer_mouse_model" value="package://twb_gazebo/meshes/computer_mouse/model.dae"/>
+  <xacro:property name="computer_mouse_model" value="package://models/meshes/computer_mouse/model.dae"/>
   <joint name="${name}_${computer_mouse}_joint" type="fixed">
     <axis xyz="0 0 1"/>
@@ -80,5 +80,5 @@
   <!--FLASH DRIVE-->
   <xacro:property name="flash_drive" value="flash_drive"/>
-  <xacro:property name="flash_drive_model" value="package://twb_gazebo/meshes/flash_drive/meshes/flash_drive.dae"/>
+  <xacro:property name="flash_drive_model" value="package://models/meshes/flash_drive/meshes/flash_drive.dae"/>
   <joint name="${name}_${flash_drive}_joint" type="fixed">
     <axis xyz="0 0 1"/>
@@ -106,5 +106,5 @@
   <!--HAND-->
   <xacro:property name="hand" value="hand"/>
-  <xacro:property name="hand_model" value="package://twb_gazebo/meshes/hand/hand.dae"/>
+  <xacro:property name="hand_model" value="package://models/meshes/hand/hand.dae"/>
   <joint name="${name}_${hand}_joint" type="fixed">
     <axis xyz="0 0 1"/>
@@ -132,5 +132,5 @@
   <!--LCD MONITOR-->
   <xacro:property name="lcd_monitor" value="lcd_monitor"/>
-  <xacro:property name="lcd_monitor_model" value="package://twb_gazebo/meshes/lcd_monitor/model.dae"/>
+  <xacro:property name="lcd_monitor_model" value="package://models/meshes/lcd_monitor/model.dae"/>
   <joint name="${name}_${lcd_monitor}_joint" type="fixed">
     <axis xyz="0 0 1"/>
@@ -158,5 +158,5 @@
   <!--MUG-->
   <xacro:property name="mug" value="mug"/>
-  <xacro:property name="mug_model" value="package://twb_gazebo/meshes/mug/meshes/mug.dae"/>
+  <xacro:property name="mug_model" value="package://models/meshes/mug/meshes/mug.dae"/>
   <joint name="${name}_${mug}_joint" type="fixed">
     <axis xyz="0 0 1"/>
@@ -184,5 +184,5 @@
   <!--NOTEPAD-->
   <xacro:property name="notepad" value="notepad"/>
-  <xacro:property name="notepad_model" value="package://twb_gazebo/meshes/notepad/meshes/notepad.dae"/>
+  <xacro:property name="notepad_model" value="package://models/meshes/notepad/meshes/notepad.dae"/>
   <joint name="${name}_${notepad}_joint" type="fixed">
     <axis xyz="0 0 1"/>
@@ -210,5 +210,5 @@
   <!--OFFICE DESK-->
   <xacro:property name="office_desk" value="office_desk"/>
-  <xacro:property name="office_desk_model" value="package://twb_gazebo/meshes/office_desk/meshes/office_desk.dae"/>
+  <xacro:property name="office_desk_model" value="package://models/meshes/office_desk/meshes/office_desk.dae"/>
   <joint name="${name}_${office_desk}_joint" type="fixed">
     <axis xyz="0 0 1"/>
@@ -236,5 +236,5 @@
   <!--PET BOTTLE-->
   <xacro:property name="pet_bottle" value="pet_bottle"/>
-  <xacro:property name="pet_bottle_model" value="package://twb_gazebo/meshes/pet_bottle/meshes/pet_bottle.dae"/>
+  <xacro:property name="pet_bottle_model" value="package://models/meshes/pet_bottle/meshes/pet_bottle.dae"/>
   <joint name="${name}_${pet_bottle}_joint" type="fixed">
     <axis xyz="0 0 1"/>
@@ -262,5 +262,5 @@
   <!--USB CABLE-->
   <xacro:property name="usb_cable" value="usb_cable"/>
-  <xacro:property name="usb_cable_model" value="package://twb_gazebo/meshes/usb_cable/model.dae"/>
+  <xacro:property name="usb_cable_model" value="package://models/meshes/usb_cable/model.dae"/>
   <joint name="${name}_${usb_cable}_joint" type="fixed">
     <axis xyz="0 0 1"/>
@@ -288,5 +288,5 @@
   <!--WORK CHAIR-->
   <xacro:property name="modern_office_chair" value="modern_office_chair"/>
-  <xacro:property name="modern_office_chair_model" value="package://twb_gazebo/meshes/modern_office_chair/model.dae"/>
+  <xacro:property name="modern_office_chair_model" value="package://models/meshes/modern_office_chair/model.dae"/>
   <joint name="${name}_${modern_office_chair}_joint" type="fixed">
     <axis xyz="0 0 1"/>

File: urdf/twb.xacro (robot description, xacro)
@@ -1,5 +1,5 @@
 <?xml version="1.0"?>
 <robot xmlns:xacro="http://www.ros.org/wiki/xacro" name="twb">
-  <xacro:property name="model_filename" value="package://twb_gazebo/meshes/twb/twb.dae"/>
+  <xacro:property name="model_filename" value="package://models/meshes/twb/twb.dae"/>
   <xacro:property name="name" value="twb"/>
   <xacro:property name="parent" value="map"/>
